File: kicad/rocinante1/rocinante1.sch (KiCad schematic (older format))
At the start: 142 parts, among them J1 ESP_01, J10 KEYBOARD, J11 SERIAL, J12 SD_Card, J13 USBFS/POWER, J14 I2S, J15 NEOPIXEL, J16 EXPHDR, J2 SWD, J3 COMPOSITE, J4 CTRL1, J5 CTRL2, J6 VGA, J7 AUDIOIN, J8 AUDIOOUT, J9 MOUSE, Q1 Q_NPN_CBE, SW1 RESET, SW2 USER1, SW3 USER2, SW4 USER3, SW5 BOOT0, U1 STM32H743IITx, U2 W9812G6KH-6, U3 LD1117S33TR_SOT223, X1 ASE-14.31818MHz, Y1 25MHz

Commit message: add background color and initial fake NTSC
Parts:
- BT1: Description resistor 1225 ohms -> 1225 coin cell battery holder
- C3, C5: Description 100 mΩ ESR, 20% tolerance -> 2.2µF, 100 mΩ ESR, 20% tolerance
- F1: Description fuse -> fuse, 16V, 100A Max, 500mA hold, 1A 100ms trip
- R9: Description Resistor 4.3Kohms 5% -> Resistor 3.4Kohms 5%
Changed lines of the file:
@@
 F 6 "Digikey" H 13075 -100 60  0001 C CNN "Distributor"
 F 7 "507-1786-1-ND" H 13075 -100 60  0001 C CNN "Distributor PN"
-F 8 "fuse" H 15025 2850 50  0001 C CNN "Description"
+F 8 "fuse, 16V, 100A Max, 500mA hold, 1A 100ms trip" H 15025 2850 50  0001 C CNN "Description"
 F 9 "1210" H 15025 2850 50  0001 C CNN "Package"
 F 10 "SMD" H 15025 2850 50  0001 C CNN "Type"
@@
 F 6 "do not place" H 7275 1200 50  0001 C CNN "Do Not Place"
 F 7 "PTH" H 7275 1200 50  0001 C CNN "Type"
-F 8 "resistor 1225 ohms" H 7275 1200 50  0001 C CNN "Description"
+F 8 "1225 coin cell battery holder" H 7275 1200 50  0001 C CNN "Description"
 	1    7275 1200
 	1    0    0    -1
@@
 F 2 "Capacitor_SMD:C_0603_1608Metric" H 850 2050 50  0001 C CNN
 F 3 "~" H 850 2050 50  0001 C CNN
-F 4 "100 mΩ ESR, 20% tolerance" V 850 2050 50  0001 C CNN "Description"
+F 4 "2.2µF, 100 mΩ ESR, 20% tolerance" V 850 2050 50  0001 C CNN "Description"
 F 5 "0603" H 12150 1900 60  0001 L CNN "Package"
 F 6 "SMD" H 850 2050 50  0001 C CNN "Type"
@@
 F 2 "Capacitor_SMD:C_0603_1608Metric" H 1025 2050 50  0001 C CNN
 F 3 "~" H 1025 2050 50  0001 C CNN
-F 4 "100 mΩ ESR, 20% tolerance" V 1025 2050 50  0001 C CNN "Description"
+F 4 "2.2µF, 100 mΩ ESR, 20% tolerance" V 1025 2050 50  0001 C CNN "Description"
 F 5 "0603" H 12150 1900 60  0001 L CNN "Package"
 F 6 "SMD" H 1025 2050 50  0001 C CNN "Type"
@@
 F 2 "Resistor_SMD:R_0603_1608Metric" V 5855 10300 50  0001 C CNN
 F 3 "" H 5925 10300 50  0001 C CNN
-F 4 "Resistor 4.3Kohms 5%" V 5925 10300 50  0001 C CNN "Description"
+F 4 "Resistor 3.4Kohms 5%" V 5925 10300 50  0001 C CNN "Description"
 F 5 "0603" H 5925 10300 50  0001 C CNN "Package"
 F 6 "SMD" H 5925 10300 50  0001 C CNN "Type"
