File: kicad/rocinante1/rocinante1.sch (KiCad schematic (older format))
At the start: 7 parts

Commit message: checkpoint schematic
Parts:
- removed C?: 10µF, symbol Device:CP1
- removed R? (x4): 68K, symbol Device:R
- removed U?: STM32F746VGHx, Package_BGA:TFBGA-100_8x8mm_Layout10x10_P0.8mm, symbol MCU_ST_STM32F7:STM32F746VGHx
- added BT1: Battery_Cell, symbol Device:Battery_Cell
- added C10, C11: 2.2µF, Capacitors_SMD:C_0805, symbol Device:C_Small
- added C13, C2, C3, C4, C7, C8, C9: 100nF, Capacitors_SMD:C_0805, symbol Device:C_Small
- added C14: 100nF, Capacitors_SMD:C_1206, symbol Device:CP1
- added C15, C22: 4.7µ, Capacitors_SMD:C_1206, symbol Device:C_Small
- added C21: 1µ, Capacitors_SMD:C_0805, symbol Device:C_Small
- added C5, C6: 22pF, Capacitors_SMD:C_0805, symbol Device:C_Small
- added D1: DEBUG LED, LEDs:LED-0805, symbol Device:LED
- added F1: F_Small, Resistors_SMD:R_1210, symbol MOBO_SMD_V2-rescue:F_Small
- added J2: USB_A, Connectors:USB_A, symbol MOBO_SMD_V2-rescue:USB_A
- added P2: USB_OTG, microusb:10118192-0001LF, symbol MOBO_SMD_V2-rescue:USB_OTG
- added R1, R4, R6, R7, R8, R9: 68K, Resistors_SMD:R_0805, symbol Device:R
- added R10, R13, R22, R23, R24, R25: 22, Resistors_SMD:R_0805, symbol Device:R
- added R12: 220, Resistors_SMD:R_0805, symbol Device:R
- added R?: 10K, symbol Device:R_US
- added SW?: SW_Push, symbol Switch:SW_Push
- added U1: STM32H745IGTx, Package_QFP:LQFP-176_24x24mm_P0.5mm, symbol STM32H745IGTx:STM32H745IGTx
- added Y2: 16MHz, Crystals:ABM3, symbol Device:Crystal
- J1: renamed from J?; footprint (none) -> Connector_Card:microSD_HC_Molex_104031-0811
Connections:
- net labels added: +3V3, +5V, BAT, BOOT, CLOCK0, CLOCK1, DEBUG_LED, SDIO_CLK, SDIO_CMD, SDIO_D0, SDIO_D1, SDIO_D2, SDIO_D3, USB_FS_D_N, USB_FS_D_P, USB_HS_D_N, USB_HS_D_P, VDD3.3
- net labels removed: SPIO_CS, SPIO_DI, SPIO_DO, SPIO_SCK
- wire segments 29 -> 118

Commit message: add most of schematic for Rosa v1
Parts:
- removed J1: Micro_SD_Card, Connector_Card:microSD_HC_Molex_104031-0811, symbol Connector:Micro_SD_Card
- removed J2: USB_A, Connectors:USB_A, symbol MOBO_SMD_V2-rescue:USB_A
- removed R?: 10K, symbol Device:R_US
- removed U1: STM32H745IGTx, Package_QFP:LQFP-176_24x24mm_P0.5mm, symbol STM32H745IGTx:STM32H745IGTx
- added C1: 1nF, Capacitors_SMD:C_0805, symbol Device:C_Small
- added C10, C12, C14, C16, C17, C18, C19, C20, C5, C8: 100nF, Capacitors_SMD:C_0805, symbol Device:C_Small
- added D2: LED2, LEDs:LED-0805, symbol Device:LED
- added D3: LED3, LEDs:LED-0805, symbol Device:LED
- added J1: RCJ-044, CUI_RCJ-044:CUI_RCJ-044, symbol RCJ-044:RCJ-044
- added J10: Conn_01x06_Male, Connector_PinHeader_2.54mm:PinHeader_1x06_P2.54mm_Vertical, symbol Connector:Conn_01x06_Male
- added J11: SD_Card, Connector_Card:SD_Kyocera_145638009511859+, symbol Connector:SD_Card
- added J2: CONN_02X05, Pin_Headers:Pin_Header_Straight_2x05_Pitch1.27mm_SMD, symbol ColecoHat2-rescue:CONN_02X05
- added J3: CTRL1, Connectors:DB9MD, symbol ColecoHat2-rescue:DB9_FEMALE_MountingHoles
- added J4: CTRL2, Connectors:DB9MD, symbol ColecoHat2-rescue:DB9_FEMALE_MountingHoles
- added J5: ESP_01, Connector_PinSocket_2.54mm:PinSocket_2x04_P2.54mm_Vertical, symbol Connector_Generic:Conn_02x04_Odd_Even
- added J6: AudioIn, Connector_Audio:Jack_3.5mm_CUI_SJ1-3535NG_Horizontal, symbol Connector:AudioJack3
- added J7: AudioOut, Connector_Audio:Jack_3.5mm_CUI_SJ1-3535NG_Horizontal, symbol Connector:AudioJack3
- added J8, J9: Mini-DIN-6, Mini_din6:Mini_din6, symbol Connector:Mini-DIN-6
- added R11, R13, R15, R17, R19, R21, R23, R25, R27, R29, R31, R33, R35, R5, R7, R9: TBP, Resistors_SMD:R_0805, symbol Device:R_Small
- added R3, R4: 220, Resistors_SMD:R_0805, symbol Device:R
- added R37, R63, R64, R65, R66: 10K, Resistors_SMD:R_0805, symbol Device:R_Small
- added R41, R42, R43, R44, R45, R46, R47, R48: 20K, Resistors_SMD:R_0805, symbol Device:R
- added R61, R62: TBD, Resistors_SMD:R_0805, symbol Device:R
- added SW1, SW3, SW4, SW5: SW_Push, Button_Switch_SMD:SW_Push_1P1T_NO_6x6mm_H9.5mm, symbol Switch:SW_Push
- added U1: AS4C4M16SA, Package_SO:TSOP-II-54_22.2x10.16mm_P0.8mm, symbol Memory_RAM:AS4C4M16SA
- added U2: STM32H743IITx, Package_QFP:LQFP-176_24x24mm_P0.5mm, symbol MCU_ST_STM32H7:STM32H743IITx
- added X1: ASE-14.31818MHz, Oscillator:Oscillator_SMD_Abracon_ASE-4Pin_3.2x2.5mm, symbol Oscillator:ASE-xxxMHz
- BT1: footprint (none) -> Battery:BatteryHolder_Keystone_3001_1x12mm
- C11: value 2.2µF -> 100nF
- C15, C22: value 4.7µ -> 100nF; footprint Capacitors_SMD:C_1206 -> Capacitors_SMD:C_0805
- C21: value 1µ -> 100nF
- C23: renamed from C14; value 100nF -> 10µF
- C25: renamed from C5; value 22pF -> TBD
- C26: renamed from C6; value 22pF -> TBD
- C4: value 100nF -> 2.2µF
- D1: value DEBUG LED -> LED1
- SW2: renamed from SW?; footprint (none) -> Button_Switch_SMD:SW_Push_1P1T_NO_6x6mm_H9.5mm
- Y1: renamed from Y2; value 16MHz -> 25MHz; Distributor PN 535-9103-1-ND -> 644-1367-1-ND; Manufacturer Abracon LLC -> NDK; PN ABM3-16.000MHZ-B2-T -> NX2016SA-25MHZ-EXS00A-CS11321
- renumbered C8 to C24, C10 to C6, P2 to P1, R12 to R2, R1 to R49, R4 to R50, R6 to R51, R7 to R52, R8 to R53, R9 to R54, R10 to R55, R13 to R56, R22 to R57, R23 to R58, R24 to R59, R25 to R60
Connections:
- net labels added: 3V3, 5V, ADC1_INP3, ADC1_INP5, AUDIO_IN_L, AUDIO_IN_R, CTS, CV0, CV1, CV2, CV3, CV4, CV5, CV6, CV7, DAC1_OUT1, DAC1_OUT2, DTR, E1, E2, ESP_CH_EN, ESP_GPIO0, ESP_GPIO2, ESP_RST, ESP_RX, ESP_TX, FIRE1, FIRE2, I2S1_SDO, I2S_CK, I2S_SDI, I2S_WS, KBD_CLK, KBD_DATA, LED1, LED2, LED3, MOUSE_CLK, MOUSE_DATA, N1, N2, NRST, QUADA1, QUADA2, QUADB1, QUADB2, RXI, S1, S2, SDRAM_A0, SDRAM_A1, SDRAM_A10, SDRAM_A11, SDRAM_A2, SDRAM_A3, SDRAM_A4, SDRAM_A5, SDRAM_A6, SDRAM_A7, SDRAM_A8, SDRAM_A9, SDRAM_BA0, SDRAM_BA1, SDRAM_D0, SDRAM_D1, SDRAM_D10, SDRAM_D11, SDRAM_D12, SDRAM_D13, SDRAM_D14, SDRAM_D15, SDRAM_D2, SDRAM_D3, SDRAM_D4, SDRAM_D5, SDRAM_D6, SDRAM_D7, SDRAM_D8, SDRAM_D9, SDRAM_NBL0, SDRAM_NBL1, SDRAM_SDCKE0, SDRAM_SDCLK, SDRAM_SDNCAS, SDRAM_SDNE0, SDRAM_SDNRAS, SDRAM_SDNWE, SJ1, SJ2, SK1, SK2, SWCLK, SWDIO, TIM2_CH1, TIM3_CH2, TXO, USART1_RX, USART1_TX, USART2_CK, USART2_RX, USART2_TX, USART3_CK, USART3_RX, USART3_TX, USER1, USER2, USER3, VCLK, VCLKEN, VGA_B0, VGA_B1, VGA_B2, VGA_B3, VGA_B4, VGA_G0, VGA_G1, VGA_G2, VGA_G3, VGA_G4, VGA_G5, VGA_R0, VGA_R1, VGA_R2, VGA_R3, VGA_R4, W1, W2
- net labels removed: DEBUG_LED, USB_HS_D_N, USB_HS_D_P, VDD3.3
- wire segments 118 -> 356
- no-connect marks 0 -> 4
Other:
- moved on the sheet: C24, C25, C26, C6, D1, F1, P1, R2, R58, R59, R60

Commit message: checkpoint PCB work; schematic getting pretty close
Parts:
- removed D2: LED2, LEDs:LED-0805, symbol Device:LED
- removed D3: LED3, LEDs:LED-0805, symbol Device:LED
- removed P1: USB_OTG, microusb:10118192-0001LF, symbol MOBO_SMD_V2-rescue:USB_OTG
- removed R11, R13, R17, R19, R21, R23, R5, R7, R9: TBP, Resistors_SMD:R_0805, symbol Device:R_Small
- removed R4: 220, Resistors_SMD:R_0805, symbol Device:R
- removed U1: AS4C4M16SA, Package_SO:TSOP-II-54_22.2x10.16mm_P0.8mm, symbol Memory_RAM:AS4C4M16SA
- added C19: 70nF, Capacitor_SMD:C_0603_1608Metric, symbol Device:C_Small
- added C2, C31, C32: 100nF, Capacitor_SMD:C_0603_1608Metric, symbol Device:C_Small
- added C26, C27: 10µF, Capacitor_THT:CP_Radial_D5.0mm_P2.00mm, symbol Device:CP1_Small
- added C33, C35: 1µF, Capacitor_THT:CP_Radial_D5.0mm_P2.00mm, symbol Device:C_Small
- added C34: 4.7µF, Capacitor_THT:CP_Radial_D5.0mm_P2.00mm, symbol Device:C_Small
- added D4: RGBLED1, LED_SMD:LED_WS2812B_PLCC4_5.0x5.0mm_P3.2mm, symbol LED:WS2812B
- added D5: RGBLED2, LED_SMD:LED_WS2812B_PLCC4_5.0x5.0mm_P3.2mm, symbol LED:WS2812B
- added D6: RGBLED3, LED_SMD:LED_WS2812B_PLCC4_5.0x5.0mm_P3.2mm, symbol LED:WS2812B
- added J13: USBFS/POWER, Connector_USB:USB_Micro-B_Amphenol_10104110_Horizontal, symbol Connector:USB_B_Micro
- added J14: I2S, Connector_PinHeader_2.54mm:PinHeader_1x06_P2.54mm_Vertical, symbol Connector:Conn_01x06_Male
- added J15: EXPHDR, Connector_PinSocket_2.54mm:PinSocket_2x04_P2.54mm_Vertical, symbol Connector_Generic:Conn_02x04_Odd_Even
- added J6: VGA, Connector_Dsub:DSUB-15-HD_Female_Horizontal_P2.29x1.98mm_EdgePinOffset3.03mm_Housed_MountingHolesOffset4.94mm, symbol Connector:DB15_Female_HighDensity_MountingHoles
- added Q1: Q_NPN_CBE, Package_TO_SOT_SMD:SOT-23, symbol Device:Q_NPN_CBE
- added R1: 220, Resistor_SMD:R_0603_1608Metric, symbol Device:R
- added R10: 6.9k, Resistor_SMD:R_0603_1608Metric, symbol ColecoHat2-rescue:R
- added R11: 14k, Resistor_SMD:R_0603_1608Metric, symbol ColecoHat2-rescue:R
- added R12: 28K, Resistor_SMD:R_0603_1608Metric, symbol ColecoHat2-rescue:R
- added R13: 47, Resistor_SMD:R_0603_1608Metric, symbol Device:R
- added R14, R16: 10K, Resistor_SMD:R_0603_1608Metric, symbol Device:R_Small
- added R24: 270, Resistor_SMD:R_0603_1608Metric, symbol Device:R_Small
- added R26, R37: 1100, Resistor_SMD:R_0603_1608Metric, symbol Device:R_Small
- added R28, R34, R39: 4.2k, Resistor_SMD:R_0603_1608Metric, symbol Device:R_Small
- added R30, R36: 560, Resistor_SMD:R_0603_1608Metric, symbol Device:R_Small
- added R32, R38: 2.1k, Resistor_SMD:R_0603_1608Metric, symbol Device:R_Small
- added R40, R41, R42: 150, Resistor_SMD:R_0603_1608Metric, symbol Device:R_Small
- added R5: 215, Resistor_SMD:R_0603_1608Metric, symbol ColecoHat2-rescue:R
- added R6: 430, Resistor_SMD:R_0603_1608Metric, symbol ColecoHat2-rescue:R
- added R7: 860, Resistor_SMD:R_0603_1608Metric, symbol ColecoHat2-rescue:R
- added R8: 1.7k, Resistor_SMD:R_0603_1608Metric, symbol ColecoHat2-rescue:R
- added R9: 3.4k, Resistor_SMD:R_0603_1608Metric, symbol ColecoHat2-rescue:R
- added U2: W9812G6KH-5, Package_SO:TSOP-II-54_22.2x10.16mm_P0.8mm, symbol Memory_RAM:W9812G6KH-5
- added U3: LD1117S33TR_SOT223, Package_TO_SOT_SMD:SOT-223-3_TabPin2, symbol Regulator_Linear:LD1117S33TR_SOT223
- BT1: value Battery_Cell -> 1225; Manufacturer (none) -> Keystone Electronics; Manufacturer PN (none) -> 3001; do not place (none) -> do not place
- C1: renamed from C2; footprint Capacitors_SMD:C_0805 -> Capacitor_SMD:C_0603_1608Metric; Note (none) -> +/- 20% tolerance
- C10, C11, C12, C13, C14, C15, C16, C17, C7, C8, C9: footprint Capacitors_SMD:C_0805 -> Capacitor_SMD:C_0603_1608Metric; Note (none) -> +/- 20% tolerance
- C18: value 100nF -> 70nF; footprint Capacitors_SMD:C_0805 -> Capacitor_SMD:C_0603_1608Metric
- C20: renamed from C1; footprint Capacitors_SMD:C_0805 -> Capacitor_SMD:C_0603_1608Metric
- C21: renamed from C19; footprint Capacitors_SMD:C_0805 -> Capacitor_SMD:C_0603_1608Metric
- C22: renamed from C20; footprint Capacitors_SMD:C_0805 -> Capacitor_SMD:C_0603_1608Metric
- C23: renamed from C21; footprint Capacitors_SMD:C_0805 -> Capacitor_SMD:C_0603_1608Metric
- C24: renamed from C22; footprint Capacitors_SMD:C_0805 -> Capacitor_SMD:C_0603_1608Metric
- C25: renamed from C23; footprint Capacitors_SMD:C_1206 -> Capacitor_THT:CP_Radial_D5.0mm_P2.00mm
- C28: renamed from C24; footprint Capacitors_SMD:C_0805 -> Capacitor_SMD:C_0603_1608Metric
- C29: renamed from C25; footprint Capacitors_SMD:C_0805 -> Capacitor_SMD:C_0603_1608Metric
- C3, C5: value 100nF -> 2.2µF; footprint Capacitors_SMD:C_0805 -> Capacitor_THT:CP_Radial_D5.0mm_P2.00mm; Note (none) -> 100 mΩ ESR, 20% tolerance
- C30: renamed from C26; footprint Capacitors_SMD:C_0805 -> Capacitor_SMD:C_0603_1608Metric
- C4, C6: value 2.2µF -> 100nF; footprint Capacitors_SMD:C_0805 -> Capacitor_SMD:C_0603_1608Metric; Note (none) -> +/- 20% tolerance
- D1: value LED1 -> POWER; footprint LEDs:LED-0805 -> LED_SMD:LED_0603_1608Metric; Color (none) -> Green
- F1: footprint Resistors_SMD:R_1210 -> Fuse:Fuse_1210_3225Metric
- J10: renamed from J9; value Mini-DIN-6 -> KEYBOARD
- J11: renamed from J10; value Conn_01x06_Male -> SERIAL
- J2: value CONN_02X05 -> SWD; footprint Pin_Headers:Pin_Header_Straight_2x05_Pitch1.27mm_SMD -> Connector_PinHeader_1.27mm:PinHeader_2x05_P1.27mm_Vertical_SMD
- J3: renamed from J1; value RCJ-044 -> COMPOSITE
- J4: renamed from J3; footprint Connectors:DB9MD -> Connector_Dsub:DSUB-9_Male_Horizontal_P2.77x2.84mm_EdgePinOffset7.70mm_Housed_MountingHolesOffset9.12mm; Description DB-9 right-angle TH -> (none); Distributor Digikey -> (none); Distributor PN 609-1481-ND -> (none); Distributor URL https://www.digikey.com/product-detail/en/D09P33E4GX00LF/60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 -> (none); Do Not Place do not place -> (none); Manufacturer Amphenol -> Assmann; Manufacturer PN D09P33E4GX00LF -> A-DS 09 A/KG-T2S; Package 9POS -> (none); Type thru-hole -> (none)
- J5: renamed from J4; footprint Connectors:DB9MD -> Connector_Dsub:DSUB-9_Male_Horizontal_P2.77x2.84mm_EdgePinOffset7.70mm_Housed_MountingHolesOffset9.12mm; Description DB-9 right-angle TH -> (none); Distributor Digikey -> (none); Distributor PN 609-1481-ND -> (none); Distributor URL https://www.digikey.com/product-detail/en/D09P33E4GX00LF/60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 -> (none); Do Not Place do not place -> (none); Manufacturer Amphenol -> Assmann; Manufacturer PN D09P33E4GX00LF -> A-DS 09 A/KG-T2S; Package 9POS -> (none); Type thru-hole -> (none)
- J9: renamed from J8; value Mini-DIN-6 -> MOUSE
- R15: value TBP -> 10K; footprint Resistors_SMD:R_0805 -> Resistor_SMD:R_0603_1608Metric
- R2: value 220 -> 2.2k; footprint Resistors_SMD:R_0805 -> Resistor_SMD:R_0603_1608Metric
- R21: renamed from R37; footprint Resistors_SMD:R_0805 -> Resistor_SMD:R_0603_1608Metric
- R22: renamed from R41; footprint Resistors_SMD:R_0805 -> Resistor_SMD:R_0603_1608Metric
- R23: renamed from R42; footprint Resistors_SMD:R_0805 -> Resistor_SMD:R_0603_1608Metric
- R25: value TBP -> 560; footprint Resistors_SMD:R_0805 -> Resistor_SMD:R_0603_1608Metric
- R27: value TBP -> 2.1k; footprint Resistors_SMD:R_0805 -> Resistor_SMD:R_0603_1608Metric
- R29, R35: value TBP -> 270; footprint Resistors_SMD:R_0805 -> Resistor_SMD:R_0603_1608Metric
- R3: value 220 -> 6.8k; footprint Resistors_SMD:R_0805 -> Resistor_SMD:R_0603_1608Metric
- R31: value TBP -> 1100; footprint Resistors_SMD:R_0805 -> Resistor_SMD:R_0603_1608Metric
- R33: value TBP -> 4.2k; footprint Resistors_SMD:R_0805 -> Resistor_SMD:R_0603_1608Metric
- R43, R44, R45, R46, R47, R48, R49, R50, R51, R52, R53, R54, R55, R56, R57, R58, R59, R60, R61, R62, R63, R64, R65, R66: footprint Resistors_SMD:R_0805 -> Resistor_SMD:R_0603_1608Metric
- SW1: value SW_Push -> RESET
- SW2: renamed from SW3; value SW_Push -> USER1
- SW3: renamed from SW4; value SW_Push -> USER2
- SW4: renamed from SW5; value SW_Push -> USER3
- SW5: renamed from SW2; value SW_Push -> BOOT0
- Y1: footprint Crystals:ABM3 -> Crystal:Crystal_SMD_2016-4Pin_2.0x1.6mm
- renumbered J5 to J1, J11 to J12, J6 to J7, J7 to J8, U2 to U1
Connections:
- net labels added: ADC3_INP2, ADC3_INP3, ADC3_INP6, ADC3_INP7, EXP01, EXP02, I2C1_SCL, I2C1_SDA, PADDLEA1, PADDLEA2, PADDLEB1, PADDLEB2, RGBLED_PWM, RGBLED_SPI, SDIO_CD, SPI6_MISO, SPI6_MOSI, SPI6_NSS_SWCTL, SPI6_SCK, TIM1_CH2, TIM4_CH1, TIM5_CH2, UART4_RX, UART4_TX, USART1_CK, USART2_CTS, USART2_RTS, VDD, VDD33USB, VDDA, VGA_BLUE, VGA_GREEN, VGA_HSYNC, VGA_ID0, VGA_ID1, VGA_ID2, VGA_ID3, VGA_RED, VGA_VSYNC, VREFP
- net labels removed: +3V3, 3V3, LED3, QUADA1, QUADA2, QUADB1, QUADB2, SJ1, SJ2, SK1, SK2, USART2_CK, VCLKEN
- wire segments 356 -> 484
- no-connect marks 4 -> 24
Other:
- note added: "Compatible with\nJim’s SPI header\nexcept added 7 and 8"
- note added: "VDD DECOUPLING"
- moved on the sheet: C1, C20, C21, C22, C23, C24, C28, C29, C30, F1, J2, J4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

Commit message: finish schematic draft; place some parts
Parts:
- removed J15: EXPHDR, Connector_PinSocket_2.54mm:PinSocket_2x04_P2.54mm_Vertical, symbol Connector_Generic:Conn_02x04_Odd_Even
- removed R16, R63, R64, R65, R66: 10K, Resistor_SMD:R_0603_1608Metric, symbol Device:R_Small
- removed R24, R29, R35: 270, Resistor_SMD:R_0603_1608Metric, symbol Device:R_Small
- removed R25, R30, R36: 560, Resistor_SMD:R_0603_1608Metric, symbol Device:R_Small
- removed R26, R31, R37: 1100, Resistor_SMD:R_0603_1608Metric, symbol Device:R_Small
- removed R27, R32, R38: 2.1k, Resistor_SMD:R_0603_1608Metric, symbol Device:R_Small
- removed R28, R33, R34, R39: 4.2k, Resistor_SMD:R_0603_1608Metric, symbol Device:R_Small
- added C36: 1µF, Capacitor_SMD:C_0603_1608Metric, symbol Device:C_Small
- added D2: DEBUGLED, LED_SMD:LED_0603_1608Metric, symbol Device:LED
- added J15: NEOPIXEL, Connector_PinHeader_2.54mm:PinHeader_1x03_P2.54mm_Vertical, symbol Connector:Conn_01x03_Male
- added J16: EXPHDR, Connector_PinHeader_2.54mm:PinHeader_2x05_P2.54mm_Vertical, symbol Connector_Generic:Conn_02x05_Odd_Even
- added R16, R36, R37, R38, R39: 10K, Resistor_SMD:R_0603_1608Metric, symbol Device:R
- added R17, R25, R31: 270, Resistor_SMD:R_0603_1608Metric, symbol Device:R
- added R18, R26, R32: 560, Resistor_SMD:R_0603_1608Metric, symbol Device:R
- added R19, R27, R33: 1100, Resistor_SMD:R_0603_1608Metric, symbol Device:R
- added R20, R28, R34: 2.2k, Resistor_SMD:R_0603_1608Metric, symbol Device:R
- added R24, R29, R35: 4.3k, Resistor_SMD:R_0603_1608Metric, symbol Device:R
- added R30: 8.6k, Resistor_SMD:R_0603_1608Metric, symbol Device:R
- added R4: 220, Resistor_SMD:R_0603_1608Metric, symbol Device:R
- BT1, J2: Package (none) -> THT
- C18, C19: Note (none) -> ceramic
- C25, C26, C27, C3, C33, C34, C35, C5: footprint Capacitor_THT:CP_Radial_D5.0mm_P2.00mm -> Capacitor_SMD:C_0603_1608Metric
- D1: value POWER -> POWERLED
- J1, J10, J11, J14, J4, J5, J9: Package (none) -> THT; do not place (none) -> do not place
- J12: footprint Connector_Card:SD_Kyocera_145638009511859+ -> Connector_FCI:10067847-001RLF
- J13: Manufacturer (none) -> Amphenol; Manufacturer PN (none) -> 10104110-0001LF
- J3: Field4 1.02 -> (none); Field5 CUI Devices -> (none); Field6 11.6 mm -> (none); Manufacturer (none) -> CUI Devices; Manufacturer PN (none) -> RCJ-044; Note: (none) -> YELLOW; Package (none) -> THT; do not place (none) -> do not place
- J6: footprint Connector_Dsub:DSUB-15-HD_Female_Horizontal_P2.29x1.98mm_EdgePinOffset3.03mm_Housed_MountingHolesOffset4.94mm -> DSUB15HD:HD15-SN-24; Manufacturer (none) -> Assmann; Manufacturer PN (none) -> AHDF15A-KG-TAXB; Package (none) -> THT; do not place (none) -> do not place
- J7: value AudioIn -> AUDIOIN; Package (none) -> THT; do not place (none) -> do not place
- J8: value AudioOut -> AUDIOOUT; Package (none) -> THT; do not place (none) -> do not place
- Q1: Note (none) -> NPN
- SW1: Manufacturer (none) -> C&K; Manufacturer PN (none) -> PTS645SM70SMTR92; Note (none) -> Or any SMT J TACTILE SPST 130-200gpf 4mm-10mm above PCB, RE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
- SW2, SW3, SW4, SW5: Manufacturer (none) -> C&K; Manufacturer PN (none) -> PTS645SM70SMTR92; Note (none) -> Or any SMT J TACTILE SPST 130-200gpf 4mm-10mm above PCB, BL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
- U2: value W9812G6KH-5 -> W9812G6KH-6; symbol Memory_RAM:W9812G6KH-5 -> Memory_RAM:W9812G6KH-6
- U3: Manufacturer (none) -> STMicroelectronics; Manufacturer PN (none) -> LD1117S33TR; Note (none) -> 5V in, 3.3V out
Connections:
- net labels added: DEBUG, EXPGPIO0, EXPGPIO1, EXPPWM, JOYSELECT, KEYSELECT, SDIO_WP
- net labels removed: EXP01, EXP02, LED1, LED2
- wire segments 484 -> 501
- no-connect marks 24 -> 18
Other:
- note added: "Compatible with\nJim’s SPI header\non pins 1-6"
- note removed: "Compatible with\nJim’s SPI header\nexcept added 7 and 8"
- moved on the sheet: C20, D1, J4, J5, R1, R2, R3

Commit message: Schematic done, THT PN chosen, working on routing
Parts:
- removed J10: KEYBOARD, Mini_din6:Mini_din6, symbol Connector:Mini-DIN-6
- removed J9: MOUSE, Mini_din6:Mini_din6, symbol Connector:Mini-DIN-6
- removed R14, R15: 10K, Resistor_SMD:R_0603_1608Metric, symbol Device:R_Small
- added H1: HOLE0, MountingHole:MountingHole_3.2mm_M3_Pad_Via, symbol Mechanical:MountingHole_Pad
- added H2: HOLE1, MountingHole:MountingHole_3.2mm_M3_Pad_Via, symbol Mechanical:MountingHole_Pad
- added H3: HOLE2, MountingHole:MountingHole_3.2mm_M3_Pad_Via, symbol Mechanical:MountingHole_Pad
- added H4: HOLE3, MountingHole:MountingHole_3.2mm_M3_Pad_Via, symbol Mechanical:MountingHole_Pad
- added J10: KEYBOARD, Mini_din6:CUI_MD-60SM, symbol MD-60SM:MD-60SM
- added J9: MOUSE, Mini_din6:CUI_MD-60SM, symbol MD-60SM:MD-60SM
- added R14, R15: 10K, Resistor_SMD:R_0603_1608Metric, symbol ColecoHat2-rescue:R
- added TP1: CPST, TestPoint:TestPoint_Keystone_5015_Micro-Minature, symbol Connector:TestPoint
- added TP2: 5V, TestPoint:TestPoint_Keystone_5015_Micro-Minature, symbol Connector:TestPoint
- added TP3: 3V3, TestPoint:TestPoint_Keystone_5015_Micro-Minature, symbol Connector:TestPoint
- added TP4: GND, TestPoint:TestPoint_Keystone_5015_Micro-Minature, symbol Connector:TestPoint
- added TP5: KBDDATA, TestPoint:TestPoint_Keystone_5015_Micro-Minature, symbol Connector:TestPoint
- added TP6: KBDCLK, TestPoint:TestPoint_Keystone_5015_Micro-Minature, symbol Connector:TestPoint
- J2: Manufacturer (none) -> Amphenol; Manufacturer PN (none) -> 20021521-00010C1LF; Package THT -> SMT
- J6: Manufacturer Assmann -> Adam Tech; Manufacturer PN AHDF15A-KG-TAXB -> HD15-SN-24
Connections:
- net labels added: AUDIO_OUT_L, AUDIO_OUT_R
- net labels removed: AUDIO_IN_L, AUDIO_IN_R
- wire segments 501 -> 512
Other:
- moved on the sheet: C21, C22, C23, C24, J2, R16, R22, R23, R37, R43, R44, R45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

Commit message: add some necessary BOM fields
Parts:
- BT1, J1, J11, J14, J16, J4, J5, J6, J7, J8: Do Not Place (none) -> do not place; Package THT -> (none); Type (none) -> PTH; do not place do not place -> (none)
- C1, C2, C4, C6, C7, C8: Description (none) -> 100nF ceramic capacitor +/- 20% tolerance; Note +/- 20% tolerance -> (none); Package (none) -> 0603
- C10, C11, C12, C13, C14, C15, C16, C17, C31, C32, C9: Description (none) -> 100nF ceramic capacitor +/- 20% tolerance; Note +/- 20% tolerance -> (none)
- C18: Description (none) -> 70nF ceramic capacitor; Note ceramic -> (none)
- C19: Description (none) -> 70 nF ceramic capacitor; Note ceramic -> (none)
- C20, C21, C22, C23, C24, C25, C26, C27, C28, C34, R43: Package (none) -> 0603
- C29: value TBD -> 5.1pF
- C3, C5: Description (none) -> 100 mΩ ESR, 20% tolerance; Note 100 mΩ ESR, 20% tolerance -> (none); Package (none) -> 0603
- C30: value TBD -> 5.1pF; Package (none) -> 0603
- D1: Color Green -> (none); Description (none) -> Green LED
- D2: Color Red -> (none); Description (none) -> Red LED
- F1: Manufacturer PN (none) -> 0ZCH0050FF2G; PN 0ZCH0050FF2G -> (none)
- J10, J9: Field4 Manufacturer recommendations -> (none); Field5 1.03 -> (none)
- J15: Do Not Place (none) -> do not place; do not place do not place -> (none)
- J2: Package SMT -> (none); Type (none) -> SMD
- J3: Description (none) -> yellow LED; Do Not Place (none) -> do not place; Note: YELLOW -> (none); Package THT -> (none); Type (none) -> PTH; do not place do not place -> (none)
- Q1: Description (none) -> NPN transistor; Note NPN -> (none)
- R10: Description (none) -> Resistor 6.9 Kohms 5%; Note 5% -> (none)
- R11: Description (none) -> Resistor 14 Kohms 5%; Note 5% -> (none)
- R12: Description (none) -> Resistor 28 Kohms 5%; Note 5% -> (none)
- R14, R15: Description (none) -> Resistor 10 Kohms 5% tolerance; Note .5% -> (none)
- R17, R25, R31: Description (none) -> Resistor 270 ohms .5% tolerance; Note .5% tolerance -> (none)
- R18, R26, R32: Description (none) -> Resistor 560 ohms 1% tolerance; Note 1% tolerance -> (none)
- R19, R27, R33: Description (none) -> Resistor 1100 ohms 1% tolerance; Note 1% tolerance -> (none)
- R20, R28, R34: Description (none) -> Resistor 2.2 Kohms 1% tolerance; Note 1% tolerance -> (none)
- R24, R29, R35: Description (none) -> Resistor 4.3 Kohms 2% tolerance; Note 2% tolerance -> (none)
- R30: Description (none) -> Resistor 8.6 Kohms 5% tolerance; Note 5% tolerance -> (none)
- R5: Description (none) -> Resistor 215 ohms .5%; Note .5% -> (none)
- R6: Description (none) -> Resistor 430 ohms 1%; Note 1% -> (none)
- R61, R62: value TBD -> 0; Description (none) -> resistor 0 ohms
- R7: Description (none) -> Resistor 860 ohms 1%; Note 1% -> (none)
- R8: Description (none) -> Resistor 1.7 Kohms 1%; Note 1% -> (none)
- R9: Description (none) -> Resistor 4.3Kohms 5%; Note 5% -> (none)
- SW1: Description (none) -> SMT J TACTILE SPST 130-200gpf 4mm-10mm above PCB, RED IF PO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; Note Or any SMT J TACTILE SPST 130-200gpf 4mm-10mm above PCB, RE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 -> (none)
- SW2, SW3, SW4: Description (none) -> SMT J TACTILE SPST 130-200gpf 4mm-10mm above PCB, BLACK IF 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; Note Or any SMT J TACTILE SPST 130-200gpf 4mm-10mm above PCB, BL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 -> (none)
- SW5: Description (none) -> SMT J TACTILE SPST 130-200gpf 4mm-10mm above PCB, BLUE IF P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; Note Or any SMT J TACTILE SPST 130-200gpf 4mm-10mm above PCB, BL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 -> (none)
- TP1, TP2, TP3, TP4, TP5, TP6: Description (none) -> SMT loop testpoint 3.2mm x 1.6mm, 2mm high; Note SMT loop testpoint 3.2mm x 1.6mm, 2mm high -> (none)
- U3: Description (none) -> LDO, 5V in, 3.3V out; Note 5V in, 3.3V out -> (none)
- X1: Digi-Key PN 535-11118-1-ND -> (none); Distributor (none) -> Digikey; Distributor PN (none) -> 535-11118-1-ND
- Y1: Manufacturer PN (none) -> NX2016SA-25MHZ-EXS00A-CS11321; PN NX2016SA-25MHZ-EXS00A-CS11321 -> (none)
