File: kicad/rocinante1/rocinante1.sch (KiCad schematic (older format))
At the start: 142 parts, among them J1 ESP_01, J10 KEYBOARD, J11 SERIAL, J12 SD_Card, J13 USBFS/POWER, J14 I2S, J15 NEOPIXEL, J16 EXPHDR, J2 SWD, J3 COMPOSITE, J4 CTRL1, J5 CTRL2, J6 VGA, J7 AUDIOIN, J8 AUDIOOUT, J9 MOUSE, Q1 Q_NPN_CBE, SW1 RESET, SW2 USER1, SW3 USER2, SW4 USER3, SW5 BOOT0, U1 STM32H743IITx, U2 W9812G6KH-6, U3 LD1117S33TR_SOT223, X1 ASE-14.31818MHz, Y1 25MHz

Commit message: make v1 PCB
Parts:
- BT1: Description (none) -> resistor 1225 ohms
- C1, C2, C3, C4, C5, C6, C7, C8, TP1, TP2, TP3, TP4, TP5, TP6: Type (none) -> SMD
- C10, C11, C12, C13, C14, C15, C16, C17, C18, C31, C32, C9, R10, R11, R12, R14, R15, R18, R19, R20, R24, R26, R27, R28, R29, R30, R32, R33, R34, R35, R6, R61, R62, R7, R8, R9: Package (none) -> 0603; Type (none) -> SMD
- C19: Description 70 nF ceramic capacitor -> 70nF ceramic capacitor; Package (none) -> 0603; Type (none) -> SMD
- C20: Description (none) -> 1nF ceramic capacitor; Type (none) -> SMD
- C21, C22, C23, C24, C28: Description (none) -> 100nF ceramic capacitor +/- 20% tolerance; Type (none) -> SMD
- C25, C26, C27: Description (none) -> 10µF capacitor; Type (none) -> SMD
- C29: Description (none) -> 5.1pF ceramic, +/- 5% tolerance; Package (none) -> 0603; Type (none) -> SMD
- C30: Description (none) -> 5.1pF ceramic, +/- 5% tolerance; Type (none) -> SMD
- C33, C35, C36: Description (none) -> 1µF capacitor; Package (none) -> 0603; Type (none) -> SMD
- C34: Description (none) -> 4.7µF capacitor; Type (none) -> SMD
- D1: Manufacturer (none) -> Wurth; Manufacturer PN (none) -> 150060GS75000; Package (none) -> 0603; Type (none) -> SMD
- D2: Manufacturer (none) -> Wurth; Manufacturer PN (none) -> 150060RS75000; Package (none) -> 0603; Type (none) -> SMD
- D4, D5, D6: Description (none) -> WS2812B; Manufacturer (none) -> Worldsemi; Manufacturer PN (none) -> WS2812B; Type (none) -> SMD
- F1: Description (none) -> fuse; Package (none) -> 1210; Type (none) -> SMD
- H1, H2, H3, H4: Description (none) -> mounting hole; Do Not Place (none) -> do not place; Type (none) -> PTH
- J1: Description (none) -> 2x4 header
- J10, J9: Description (none) -> MINI-DIN6; Do Not Place (none) -> do not place; Type (none) -> PTH
- J11, J14: Description (none) -> 1x6 header
- J12: Description (none) -> SD card socket; Manufacturer (none) -> Amphenol/FCI; Manufacturer PN (none) -> 10067847-001RLF; Type (none) -> SMD
- J13: Description (none) -> USB Micro B; Manufacturer Amphenol -> Amphenol/FCI; Type (none) -> SMD
- J15: Description (none) -> 1x3 header; Type (none) -> PTH
- J16: Description (none) -> 2x5 header
- J2: Description (none) -> 2x5 1.27mm header
- J3: Description yellow LED -> yellow RCA/Phono jack
- J4, J5: Description (none) -> DB9 Female
- J6: Description (none) -> DB15HD
- J7, J8: Description (none) -> 3.5mm stereo jack
- Q1: footprint Package_TO_SOT_SMD:SOT-23 -> Package_TO_SOT_SMD:SOT-323_SC-70; Manufacturer (none) -> ON Semiconductor; Manufacturer PN (none) -> MMBT3904WT1G; Package (none) -> SOT-323_SC-70; Type (none) -> SMD
- R1, R4: Description (none) -> resistor 220 ohms; Package (none) -> 0603; Type (none) -> SMD
- R13: Description (none) -> resistor 47 ohms 5%; Package (none) -> 0603; Type (none) -> SMD
- R16, R21, R36, R37, R38, R39: Description (none) -> Resistor 10 Kohms 5% tolerance; Package (none) -> 0603; Type (none) -> SMD
- R17, R25, R31: Description Resistor 270 ohms .5% tolerance -> Resistor 270 ohms 0.5% tolerance; Package (none) -> 0603; Type (none) -> SMD
- R2: Description (none) -> resistor 2.2K 5%; Package (none) -> 0603; Type (none) -> SMD
- R22, R23, R44, R45, R46, R47, R48: Description (none) -> Resistor 20 Kohms 5% tolerance; Package (none) -> 0603; Type (none) -> SMD
- R3: Description (none) -> Resistor 6.8K 5%; Package (none) -> 0603; Type (none) -> SMD
- R40, R41, R42: Description (none) -> resistor 150 ohms 5%; Package (none) -> 0603; Type (none) -> SMD
- R43: Description (none) -> Resistor 20 Kohms 5% tolerance; Type (none) -> SMD
- R49, R50, R51, R52, R53, R54: Description (none) -> Resistor 68 Kohms 5% tolerance; Package (none) -> 0603; Type (none) -> SMD
- R5: Description Resistor 215 ohms .5% -> Resistor 215 ohms 0.5%; Package (none) -> 0603; Type (none) -> SMD
- R55, R56, R57, R58, R59, R60: Description (none) -> resistor 22 ohms 5%; Package (none) -> 0603; Type (none) -> SMD
- SW1: Description SMT J TACTILE SPST 130-200gpf 4mm-10mm above PCB, RED IF PO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 -> SMT J TACTILE SPST 130-200gpf 4mm-10mm above PCB; Type (none) -> SMD
- SW2, SW3, SW4: Description SMT J TACTILE SPST 130-200gpf 4mm-10mm above PCB, BLACK IF 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 -> SMT J TACTILE SPST 130-200gpf 4mm-10mm above PCB; Type (none) -> SMD
- SW5: Description SMT J TACTILE SPST 130-200gpf 4mm-10mm above PCB, BLUE IF P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 -> SMT J TACTILE SPST 130-200gpf 4mm-10mm above PCB; Type (none) -> SMD
- U1: Description (none) -> STM32H743IITx; Manufacturer (none) -> STMicroelectronics; Manufacturer PN (none) -> STM32H743IIT6; Package (none) -> LQFP-176; Type (none) -> SMD
- U2: Description (none) -> 128MB 167MHz TSOP-II-54 SDRAM; Manufacturer (none) -> Winbond; Manufacturer PN (none) -> W9812G6KH-6; Package (none) -> TSOP-II-54; Type (none) -> SMD
- U3: Package (none) -> SOT-223-3; Type (none) -> SMD
- X1: Description (none) -> Oscillator 14.31818MHz; Package (none) -> ASE-4Pin; Type (none) -> SMD
- Y1: Description (none) -> Resonator 25MHz; Package (none) -> 2016-4pin; Type (none) -> SMD
Connections:
- wire segments 512 -> 511

Commit message: fix cap at composite out
Connections:
- wire segments 511 -> 512
Other:
- moved on the sheet: C20
Changed lines of the file:
@@
 L RCJ-044:RCJ-044 J3
 U 1 1 5F5089A0
-P 6825 10300
-F 0 "J3" H 6495 10254 50  0000 R CNN
-F 1 "COMPOSITE" H 6495 10345 50  0000 R CNN
-F 2 "CUI_RCJ-044:CUI_RCJ-044" H 6825 10300 50  0001 L BNN
-F 3 "Manufacturer Recommendations" H 6825 10300 50  0001 L BNN
-F 4 "CUI Devices" H 6825 10300 50  0001 L BNN "Manufacturer"
-F 5 "RCJ-044" H 6825 10300 50  0001 L BNN "Manufacturer PN"
-F 6 "yellow RCA/Phono jack" H 6825 10300 50  0001 C CNN "Description"
-F 7 "do not place" H 6825 10300 50  0001 C CNN "Do Not Place"
-F 8 "PTH" H 6825 10300 50  0001 C CNN "Type"
-	1    6825 10300
+P 6950 10300
+F 0 "J3" H 6620 10254 50  0000 R CNN
+F 1 "COMPOSITE" H 6620 10345 50  0000 R CNN
+F 2 "CUI_RCJ-044:CUI_RCJ-044" H 6950 10300 50  0001 L BNN
+F 3 "Manufacturer Recommendations" H 6950 10300 50  0001 L BNN
+F 4 "CUI Devices" H 6950 10300 50  0001 L BNN "Manufacturer"
+F 5 "RCJ-044" H 6950 10300 50  0001 L BNN "Manufacturer PN"
+F 6 "yellow RCA/Phono jack" H 6950 10300 50  0001 C CNN "Description"
+F 7 "do not place" H 6950 10300 50  0001 C CNN "Do Not Place"
+F 8 "PTH" H 6950 10300 50  0001 C CNN "Type"
+	1    6950 10300
 	-1   0    0    -1
 $EndComp
-$Comp
-L Device:C_Small C20
-U 1 1 5F5089A6
-P 6325 10650
-F 0 "C20" H 6417 10696 50  0000 L CNN
-F 1 "1nF" H 6417 10605 50  0000 L CNN
-F 2 "Capacitor_SMD:C_0603_1608Metric" H 6325 10650 50  0001 C CNN
-F 3 "~" H 6325 10650 50  0001 C CNN
-F 4 "0603" H 12150 1900 60  0001 L CNN "Package"
-F 5 "1nF ceramic capacitor" H 6325 10650 50  0001 C CNN "Description"
-F 6 "SMD" H 6325 10650 50  0001 C CNN "Type"
-	1    6325 10650
-	1    0    0    -1
-$EndComp
 Wire Wire Line
 	6175 10200 6325 10200
@@
 Wire Wire Line
 	6425 2750 6600 2750
-Wire Wire Line
-	6325 10750 6325 10850
 $Comp
 L ColecoHat2-rescue:R R5
@@
 $EndComp
 Connection ~ 6325 10200
+$Comp
+L Device:C_Small C20
+U 1 1 5F5089A6
+P 6325 10300
+F 0 "C20" H 6417 10346 50  0000 L CNN
+F 1 "1nF" H 6417 10255 50  0000 L CNN
+F 2 "Capacitor_SMD:C_0603_1608Metric" H 6325 10300 50  0001 C CNN
+F 3 "~" H 6325 10300 50  0001 C CNN
+F 4 "0603" H 12150 1550 60  0001 L CNN "Package"
+F 5 "1nF ceramic capacitor" H 6325 10300 50  0001 C CNN "Description"
+F 6 "SMD" H 6325 10300 50  0001 C CNN "Type"
+	1    6325 10300
+	1    0    0    -1
+$EndComp
+Wire Wire Line
+	6325 10200 6450 10200
+Wire Wire Line
+	6325 10400 6450 10400
 Wire Wire Line
-	6325 10550 6325 10400
+	6325 10400 6325 10850
+Connection ~ 6325 10400
 $EndSCHEMATC
